Commit message: Add lighthouse-based demo

File: servo_hardware_demo/urdf/servo_controller.urdf.xacro (robot description, xacro)
@@ -2,5 +2,5 @@
 <robot xmlns:xacro="http://www.ros.org/wiki/xacro" name="servo_controller">
   <!-- Include ros2_control configuration -->
-  <xacro:include filename="$(find servo_hardware_test)/urdf/servo_controller_ros_control.urdf.xacro" />
+  <xacro:include filename="$(find servo_hardware_demo)/urdf/servo_controller_ros_control.urdf.xacro" />
   <!-- Material definitions -->
   <material name="servo_body_color">

File: servo_hardware_demo/urdf/servo_controller_ros_control.urdf.xacro (robot description, xacro)
@@ -25,12 +25,4 @@
         <state_interface name="position"/>
       </joint>
-      <joint name="joint_2">
-        <command_interface name="position"/>
-        <state_interface name="position"/>
-      </joint>
-      <joint name="joint_3">
-        <command_interface name="position"/>
-        <state_interface name="position"/>
-      </joint>
     </ros2_control>
   </xacro:macro>
